Commit message: World with room and camera setup.

File: src/2020_vision/worlds/big_room.xacro (robot description, xacro)
@@ -1,3 +1,3 @@
-<sdf version='1.6'>
+<?xml version='1.0' ?>
   <world name='default'>
     <light name='sun' type='directional'>
@@ -1726,10 +1726,8 @@
       <uri>model://realsense_camera</uri>
     </include-->
-    <!-- Import macro for realsense-RS200 camera-->
     <xacro:include filename="$(find realsense_gazebo_plugin)/urdf/realsense-RS200.macro.xacro"/>
-    <!-- Create camera instance -->
-    <xacro:realsense-rs200>
-        <origin xyz="0 0 1.0" rpy="0 0 0" />
-    </xacro:realsense-rs200>
+    <xacro:realsense-d435i prefix="bottom_" parent="link">
+    <origin xyz="0.0799 0 -0.0782" rpy="0 1.5708 0" />
+  </xacro:realsense-d435i>
   </world>
 </sdf>
