Commit message: Remove floor and wall from pointcloud.

File: src/realsense_gazebo_plugin/urdf/multi_cam_2020_viz.xacro (robot description, xacro)
@@ -6,11 +6,11 @@
     <!-- Create two camera instances -->
     <xacro:realsense-rs200 prefix="first_" parent="world">
-        <origin xyz="0.4 0.4 2.3" rpy="0 0.3927 0.7854" />
+        <origin xyz="0.4 0.4 1" rpy="0 0 0.7854" />
     </xacro:realsense-rs200>
     <xacro:realsense-rs200 prefix="second_" parent="world">
-        <origin xyz="0.4 9.6 2.3" rpy="0 0.3927 -0.7854" />
+        <origin xyz="0.4 9.6 1" rpy="0 0 -0.7854" />
     </xacro:realsense-rs200>
     <xacro:realsense-rs200 prefix="third_" parent="world">
-        <origin xyz="9.6 9.6 2.3" rpy="0 0.3927 3.927" />
+        <origin xyz="9.6 9.6 1" rpy="0 0 3.927" />
     </xacro:realsense-rs200>
 </robot>
